File: breakout_board/breakout_board.sch (KiCad schematic (older format))
At the start: 13 parts, among them J1 FrontPanel, J2 USB, J3 UART, J4 OUT, J5 Conn_01x02, SW1 Reset, SW2 Boot, U1 AMS1117-3.3, U2 ESP32-S2-WROOM

Commit message: HTTP control with Web UI
Parts:
- U2: symbol ESP32-S2-WROOM:ESP32-S2-WROOM -> breakout_board-rescue:ESP32-S2-WROOM-ESP32-S2-WROOM
Changed lines of the file:
@@
 $EndComp
 $Comp
-L ESP32-S2-WROOM:ESP32-S2-WROOM U2
+L breakout_board-rescue:ESP32-S2-WROOM-ESP32-S2-WROOM U2
 U 1 1 61C57599
 P 5900 2950
