File: breakout_board/breakout_board.kicad_pcb (KiCad board)
At the start: 2 copper layers, 13 parts, among them J1 FrontPanel, J2 USB, J3 UART, J4 OUT, J5 Conn_01x02, SW1 Reset, SW2 Boot, U1 AMS1117-3.3, U2 ESP32-S2-WROOM

Commit message: New breakout board design
Parts:
- moved J2 2.84 mm to (119.4, 138.4)
- moved R1 1.80 mm to (116.8, 94.0)
- moved C2 1.80 mm to (109.2, 80.0)
- moved J1 1.80 mm to (101.6, 130.8)
- moved C1 1.80 mm to (109.2, 99.1)
- moved C3 1.80 mm to (119.4, 99.1)
- moved J3 1.80 mm to (127.0, 113.0)
- moved J4 1.80 mm to (127.0, 123.2)
- moved J5 1.80 mm to (101.6, 78.7)
- moved SW1 1.80 mm to (123.2, 90.2)
- moved SW2 1.80 mm to (123.2, 81.3)
- moved U1 1.80 mm to (109.2, 89.6)
- moved U2 1.80 mm to (105.4, 103.0)
Routing:
- net GND: track 198.6 -> 203.6 mm
- net Net-(J2-Pad2): track 3.50 -> 4.77 mm
- net Net-(J2-Pad3): track 3.78 -> 5.05 mm
- added copper zone on F.Cu, net (none)
